Commit message: setup localization

File: float_rise_description/urdf/base.urdf (robot description, URDF)
Before this commit: robot float_rise, 9 links, 8 joints
Joints:
- joint dvl_sf_joint: origin xyz=0.05 0.0 0.0 rpy=0.0 -1.5707963 0.0 -> xyz=0.0 0.0 -0.06 rpy=0.0 0.0 0.0
- joint gps_joint: origin xyz=-0.63 0.0 -0.1 rpy=0.0 0.0 0.0 -> xyz=0.075 0.0 0.635 rpy=3.1415926 0.0 0.0
- joint heave_bow_thruster_joint: origin xyz=-0.1 0.11 0.0 rpy=0.0 0.0 0.0 -> xyz=0.0 -0.11 0.08 rpy=0.0 -1.57079632679 0.0
- joint imu_sf_joint: origin xyz=-0.17 0.0 0.0 rpy=0.0 1.5707 0.0 -> xyz=0.0 0.0 0.17 rpy=0.0 0.0 0.0
- joint pressure_joint: origin xyz=0.05 0.0 0.0 rpy=0.0 0.0 0.0 -> xyz=0.00 0.0 -0.02 rpy=3.1415926 0.0 0.0
- joint surge_thruster_joint: origin xyz=-0.1 -0.11 0.0 rpy=0.0 0.0 0.0 -> xyz=0.0 0.11 0.08 rpy=0.0 -1.57079632679 0.0

Commit message: disbale the DVL

File: float_rise_description/urdf/base.urdf (robot description, URDF)
Before this commit: robot float_rise, 9 links, 8 joints
Links:
- removed link dvl_sf
Joints:
- removed joint dvl_sf_joint

Commit message: add readme

File: float_rise_description/urdf/base.urdf (robot description, URDF)
Before this commit: robot float_rise, 8 links, 7 joints
Links:
- added link usbl
Joints:
- added joint usbl_joint: type fixed, parent base_link, child usbl, origin xyz=0.0 0.0 -0.06 rpy=0.0 0.0 0.0
