Commit message: add odometry in URDF

File: float_rise_description/urdf/float_1/base.urdf (robot description, URDF)
Before this commit: robot float_rise, 9 links, 8 joints
Links:
- added link odometry_sf
Joints:
- added joint odometry_sf_joint: type fixed, parent base_link, child odometry_sf, origin xyz=0.0 0.0 0.00 rpy=3.1415926 0.0 0.0

File: float_rise_description/urdf/float_2/base.urdf (robot description, URDF)
Before this commit: robot float_rise, 9 links, 8 joints
Links:
- added link odometry_sf
Joints:
- added joint odometry_sf_joint: type fixed, parent base_link, child odometry_sf, origin xyz=0.0 0.0 0.00 rpy=3.1415926 0.0 0.0

File: float_rise_description/urdf/float_3/base.urdf (robot description, URDF)
Before this commit: robot float_rise, 8 links, 7 joints
Links:
- added link odometry_sf
Joints:
- added joint odometry_sf_joint: type fixed, parent base_link, child odometry_sf, origin xyz=0.0 0.0 0.00 rpy=3.1415926 0.0 0.0

Commit message: add acoustic sensors for floats

File: float_rise_description/urdf/float_1/base.urdf (robot description, URDF)
Before this commit: robot float_rise, 10 links, 9 joints
Links:
- removed link usbl
- added link acomm_21
- added link acomm_31
- added link usbl_12
- added link usbl_13
Joints:
- removed joint usbl_joint
- added joint acomm_21_joint: type fixed, parent base_link, child acomm_21, origin xyz=0.0 0.0 -0.06 rpy=0.0 0.0 0.0
- added joint acomm_31_joint: type fixed, parent base_link, child acomm_31, origin xyz=0.0 0.0 -0.06 rpy=0.0 0.0 0.0
- added joint usbl_12_joint: type fixed, parent base_link, child usbl_12, origin xyz=0.0 0.0 -0.06 rpy=0.0 0.0 0.0
- added joint usbl_13_joint: type fixed, parent base_link, child usbl_13, origin xyz=0.0 0.0 -0.06 rpy=0.0 0.0 0.0

File: float_rise_description/urdf/float_2/base.urdf (robot description, URDF)
Before this commit: robot float_rise, 10 links, 9 joints
Links:
- removed link acomm
- added link acomm_12
- added link acomm_32
- added link usbl_21
- added link usbl_23
Joints:
- removed joint acomm_joint
- added joint acomm_12_joint: type fixed, parent base_link, child acomm_12, origin xyz=0.0 0.0 -0.06 rpy=0.0 0.0 0.0
- added joint acomm_32_joint: type fixed, parent base_link, child acomm_32, origin xyz=0.0 0.0 -0.06 rpy=0.0 0.0 0.0
- added joint usbl_21_joint: type fixed, parent base_link, child usbl_21, origin xyz=0.0 0.0 -0.06 rpy=0.0 0.0 0.0
- added joint usbl_23_joint: type fixed, parent base_link, child usbl_23, origin xyz=0.0 0.0 -0.06 rpy=0.0 0.0 0.0

File: float_rise_description/urdf/float_3/base.urdf (robot description, URDF)
Before this commit: robot float_rise, 9 links, 8 joints
Links:
- added link acomm_13
- added link acomm_23
- added link usbl_31
- added link usbl_32
Joints:
- added joint acomm_13_joint: type fixed, parent base_link, child acomm_13, origin xyz=0.0 0.0 -0.06 rpy=0.0 0.0 0.0
- added joint acomm_23_joint: type fixed, parent base_link, child acomm_23, origin xyz=0.0 0.0 -0.06 rpy=0.0 0.0 0.0
- added joint usbl_31_joint: type fixed, parent base_link, child usbl_31, origin xyz=0.0 0.0 -0.06 rpy=0.0 0.0 0.0
- added joint usbl_32_joint: type fixed, parent base_link, child usbl_32, origin xyz=0.0 0.0 -0.06 rpy=0.0 0.0 0.0

Commit message: launch individual floats 1-5

File: float_rise_description/urdf/float_1/base.urdf (robot description, URDF)
Before this commit: robot float_rise, 13 links, 12 joints
Links:
- removed link acomm_21
- removed link acomm_31
- removed link usbl_12
- removed link usbl_13
Joints:
- removed joint acomm_21_joint
- removed joint acomm_31_joint
- removed joint usbl_12_joint
- removed joint usbl_13_joint

File: float_rise_description/urdf/float_2/base.urdf (robot description, URDF)
Before this commit: robot float_rise, 13 links, 12 joints
Links:
- removed link acomm_12
- removed link acomm_32
- removed link usbl_21
- removed link usbl_23
Joints:
- removed joint acomm_12_joint
- removed joint acomm_32_joint
- removed joint usbl_21_joint
- removed joint usbl_23_joint

Commit message: finish

File: float_rise_description/urdf/float_1/base.urdf (robot description, URDF)
Before this commit: robot float_rise, 9 links, 8 joints
Links:
- added link dvl_sf
Joints:
- added joint dvl_sf_joint: type fixed, parent base_link, child dvl_sf, origin xyz=0.0 0.0 -0.06 rpy=0.0 0.0 0.0

File: float_rise_description/urdf/float_10/base.urdf (robot description, URDF)
Before this commit: robot float_rise, 9 links, 8 joints
Links:
- added link dvl_sf
Joints:
- added joint dvl_sf_joint: type fixed, parent base_link, child dvl_sf, origin xyz=0.0 0.0 -0.06 rpy=0.0 0.0 0.0

File: float_rise_description/urdf/float_2/base.urdf (robot description, URDF)
Before this commit: robot float_rise, 9 links, 8 joints
Links:
- added link dvl_sf
Joints:
- added joint dvl_sf_joint: type fixed, parent base_link, child dvl_sf, origin xyz=0.0 0.0 -0.06 rpy=0.0 0.0 0.0

File: float_rise_description/urdf/float_3/base.urdf (robot description, URDF)
Before this commit: robot float_rise, 9 links, 8 joints
Links:
- added link dvl_sf
Joints:
- added joint dvl_sf_joint: type fixed, parent base_link, child dvl_sf, origin xyz=0.0 0.0 -0.06 rpy=0.0 0.0 0.0
